Commit message: sensor was wrongly positioned in the baseframe

File: micro_epsilon_scancontrol_description/urdf/scancontrol_30xx_25_macro.xacro (robot description, xacro)
@@ -1,9 +1,9 @@
 <?xml version="1.0" ?>
 <robot xmlns:xacro="http://wiki.ros.org/xacro">
-  <!-- Macro for both 26x0 and 29x0 - 25 scan control sensor productlines -->
+  <!-- Macro for 30xx_25 scan control sensors  -->
   <xacro:macro name="microepsilon_scancontrol_30xx_25" params="prefix">
     <link name="${prefix}base_link">
       <visual>
-        <origin xyz="0.0205 -0.0345 0" rpy="${pi/2} 0 ${pi}"/>
+        <origin xyz="-0.0435 0.0 0.0" rpy="${pi/2} 0 ${pi}"/>
         <geometry>
           <mesh filename="package://micro_epsilon_scancontrol_description/meshes/visual/visual_30xx_25.dae"/>
@@ -14,5 +14,5 @@
       </visual>
       <collision>
-        <origin xyz="0.0205 0.0345 0" rpy="${pi/2} 0 ${pi}"/>
+        <origin xyz="-0.0435 0.0 0.0" rpy="${pi/2} 0 ${pi}"/>
         <geometry>
           <mesh filename="package://micro_epsilon_scancontrol_description/meshes/collision/collision_30xx_25.stl"/>

Commit message: updated meshes for 30xx so it`s more logically positioned and does not include faces that show the measurement range.

File: micro_epsilon_scancontrol_description/urdf/scancontrol_30xx_25_macro.xacro (robot description, xacro)
@@ -5,5 +5,5 @@
     <link name="${prefix}base_link">
       <visual>
-        <origin xyz="-0.0435 0.0 0.0" rpy="${pi/2} 0 ${pi}"/>
+        <origin xyz="0.0 0.0 0.0" rpy="0 0 0"/>
         <geometry>
           <mesh filename="package://micro_epsilon_scancontrol_description/meshes/visual/visual_30xx_25.dae"/>
@@ -14,5 +14,5 @@
       </visual>
       <collision>
-        <origin xyz="-0.0435 0.0 0.0" rpy="${pi/2} 0 ${pi}"/>
+        <origin xyz="0 0.0 0.0" rpy="0 0 0"/>
         <geometry>
           <mesh filename="package://micro_epsilon_scancontrol_description/meshes/collision/collision_30xx_25.stl"/>
@@ -22,5 +22,7 @@
     <link name="${prefix}aperture_frame" />
     <joint name="${prefix}base_link-${prefix}aperture_frame" type="fixed">
-      <origin xyz="0 0 0" rpy="${pi} 0 ${pi/2}" />
+     <!-- xyz values represent the distance between the top mounting hole and the lens of the laser  -->
+     <!-- rpy values are chosen so the x and z axes are consistent with the internal sensor measurement frame -->
+      <origin xyz="-0.0935 0 -0.0767" rpy="${pi} 0 ${pi/2}" />
       <parent link="${prefix}base_link" />
       <child link="${prefix}aperture_frame" />
