Commit message: description pkg working

File: micro_epsilon_scancontrol_description/urdf/scancontrol_26x0_29x0_25_macro.xacro (robot description, xacro)
@@ -7,5 +7,5 @@
         <origin xyz="0 0 0" rpy="${pi/2} 0 ${pi/2}"/>
         <geometry>
-          <mesh filename="package://micro_epsilon_scancontrol_description/meshes/visual/visual.dae"/>
+          <mesh filename="package://micro_epsilon_scancontrol_description/meshes/visual/26x0_29x0_25.dae"/>
        </geometry>
        <material name="microepsilon_silver">
@@ -16,5 +16,5 @@
         <origin xyz="0 0 0" rpy="${pi/2} 0 ${pi/2}"/>
         <geometry>
-          <mesh filename="package://micro_epsilon_scancontrol_description/meshes/collision/collision.stl"/>
+          <mesh filename="package://micro_epsilon_scancontrol_description/meshes/collision/26x0_29x0_25.stl"/>
         </geometry>
       </collision>
