Commit message: Rename mesh files
Inconsistent naming between files and duplication of folder name(s).

File: micro_epsilon_scancontrol_description/urdf/scancontrol_27x0_100_macro.xacro (robot description, xacro)
@@ -7,5 +7,5 @@
         <origin xyz="0.0205 -0.0345 0" rpy="${pi/2} 0 ${pi}"/>
         <geometry>
-          <mesh filename="package://micro_epsilon_scancontrol_description/meshes/visual/visual_27x0_100.dae"/>
+          <mesh filename="package://micro_epsilon_scancontrol_description/meshes/visual/27x0_100.dae"/>
        </geometry>
        <material name="microepsilon_silver">
@@ -16,5 +16,5 @@
         <origin xyz="0.0205 0.0345 0" rpy="${pi/2} 0 ${pi}"/>
         <geometry>
-          <mesh filename="package://micro_epsilon_scancontrol_description/meshes/collision/collision_27x0_100.stl"/>
+          <mesh filename="package://micro_epsilon_scancontrol_description/meshes/collision/27x0_100.stl"/>
         </geometry>
       </collision>

File: micro_epsilon_scancontrol_description/urdf/scancontrol_30xx_25_macro.xacro (robot description, xacro)
@@ -7,5 +7,5 @@
         <origin xyz="0.0 0.0 0.0" rpy="0 0 0"/>
         <geometry>
-          <mesh filename="package://micro_epsilon_scancontrol_description/meshes/visual/visual_30xx_25.dae"/>
+          <mesh filename="package://micro_epsilon_scancontrol_description/meshes/visual/30xx_25.dae"/>
        </geometry>
        <material name="microepsilon_silver">
@@ -16,5 +16,5 @@
         <origin xyz="0 0.0 0.0" rpy="0 0 0"/>
         <geometry>
-          <mesh filename="package://micro_epsilon_scancontrol_description/meshes/collision/collision_30xx_25.stl"/>
+          <mesh filename="package://micro_epsilon_scancontrol_description/meshes/collision/30xx_25.stl"/>
         </geometry>
       </collision>
