Commit message: Update naming conventions and add launch tests

File: micro_epsilon_scancontrol_support/urdf/26x0_29x0_25_macro.xacro (robot description, xacro)
@@ -2,10 +2,10 @@
 <robot xmlns:xacro="http://wiki.ros.org/xacro">
   <!-- Macro for both 26x0 and 29x0 - 25 scan control sensor productlines -->
-  <xacro:macro name="microepsilon_scancontrol_26x0_29x0_25" params="prefix">
+  <xacro:macro name="micro_epsilon_scancontrol_26x0_29x0_25" params="prefix">
     <link name="${prefix}base_link">
       <visual>
         <origin xyz="0 0 0" rpy="${pi/2} 0 ${pi/2}"/>
         <geometry>
-          <mesh filename="package://micro_epsilon_scancontrol_description/meshes/visual/visual.dae"/>
+          <mesh filename="package://micro_epsilon_scancontrol_support/meshes/26x0_29x0_25/visual/base_link.dae"/>
        </geometry>
        <material name="microepsilon_silver">
@@ -16,5 +16,5 @@
         <origin xyz="0 0 0" rpy="${pi/2} 0 ${pi/2}"/>
         <geometry>
-          <mesh filename="package://micro_epsilon_scancontrol_description/meshes/collision/collision.stl"/>
+          <mesh filename="package://micro_epsilon_scancontrol_support/meshes/26x0_29x0_25/collision/base_link.stl"/>
         </geometry>
       </collision>

File: micro_epsilon_scancontrol_support/urdf/27x0_100_macro.xacro (robot description, xacro)
@@ -2,10 +2,10 @@
 <robot xmlns:xacro="http://wiki.ros.org/xacro">
   <!-- Macro for both 26x0 and 29x0 - 25 scan control sensor productlines -->
-  <xacro:macro name="microepsilon_scancontrol_27x0_100" params="prefix">
+  <xacro:macro name="micro_epsilon_scancontrol_27x0_100" params="prefix">
     <link name="${prefix}base_link">
       <visual>
         <origin xyz="0.0205 -0.0345 0" rpy="${pi/2} 0 ${pi}"/>
         <geometry>
-          <mesh filename="package://micro_epsilon_scancontrol_description/meshes/visual/visual_27x0_100.dae"/>
+          <mesh filename="package://micro_epsilon_scancontrol_support/meshes/27x0_100/visual/base_link.dae"/>
        </geometry>
        <material name="microepsilon_silver">
@@ -16,5 +16,5 @@
         <origin xyz="0.0205 0.0345 0" rpy="${pi/2} 0 ${pi}"/>
         <geometry>
-          <mesh filename="package://micro_epsilon_scancontrol_description/meshes/collision/collision_27x0_100.stl"/>
+          <mesh filename="package://micro_epsilon_scancontrol_support/meshes/27x0_100/collision/base_link.stl"/>
         </geometry>
       </collision>

File: micro_epsilon_scancontrol_support/urdf/30x0_25_macro.xacro (robot description, xacro)
@@ -2,10 +2,10 @@
 <robot xmlns:xacro="http://wiki.ros.org/xacro">
   <!-- Macro for 30xx_25 scan control sensors  -->
-  <xacro:macro name="microepsilon_scancontrol_30xx_25" params="prefix">
+  <xacro:macro name="micro_epsilon_scancontrol_30x0_25" params="prefix">
     <link name="${prefix}base_link">
       <visual>
         <origin xyz="0.0 0.0 0.0" rpy="0 0 0"/>
         <geometry>
-          <mesh filename="package://micro_epsilon_scancontrol_description/meshes/visual/visual_30xx_25.dae"/>
+          <mesh filename="package://micro_epsilon_scancontrol_support/meshes/30x0_25/visual/base_link.dae"/>
        </geometry>
        <material name="microepsilon_silver">
@@ -16,5 +16,5 @@
         <origin xyz="0 0.0 0.0" rpy="0 0 0"/>
         <geometry>
-          <mesh filename="package://micro_epsilon_scancontrol_description/meshes/collision/collision_30xx_25.stl"/>
+          <mesh filename="package://micro_epsilon_scancontrol_support/meshes/30x0_25/collision/base_link.stl"/>
         </geometry>
       </collision>

Commit message: Update default frame_id and topic name

File: micro_epsilon_scancontrol_support/urdf/26x0_29x0_25_macro.xacro (robot description, xacro)
@@ -20,9 +20,9 @@
       </collision>
     </link>
-    <link name="${prefix}aperture_frame" />
-    <joint name="${prefix}base_link-${prefix}aperture_frame" type="fixed">
+    <link name="${prefix}optical_frame" />
+    <joint name="${prefix}base_link-optical_frame" type="fixed">
       <origin xyz="0 0 0" rpy="${pi} 0 ${pi/2}" />
       <parent link="${prefix}base_link" />
-      <child link="${prefix}aperture_frame" />
+      <child link="${prefix}optical_frame" />
     </joint>
   </xacro:macro>

File: micro_epsilon_scancontrol_support/urdf/27x0_100_macro.xacro (robot description, xacro)
@@ -20,9 +20,9 @@
       </collision>
     </link>
-    <link name="${prefix}aperture_frame" />
-    <joint name="${prefix}base_link-${prefix}aperture_frame" type="fixed">
+    <link name="${prefix}optical_frame" />
+    <joint name="${prefix}base_link-optical_frame" type="fixed">
       <origin xyz="0 0 0" rpy="${pi} 0 ${pi/2}" />
       <parent link="${prefix}base_link" />
-      <child link="${prefix}aperture_frame" />
+      <child link="${prefix}optical_frame" />
     </joint>
   </xacro:macro>

File: micro_epsilon_scancontrol_support/urdf/30x0_25_macro.xacro (robot description, xacro)
@@ -20,11 +20,11 @@
       </collision>
     </link>
-    <link name="${prefix}aperture_frame" />
-    <joint name="${prefix}base_link-${prefix}aperture_frame" type="fixed">
+    <link name="${prefix}optical_frame" />
+    <joint name="${prefix}base_link-optical_frame" type="fixed">
      <!-- xyz values represent the distance between the top mounting hole and the lens of the laser  -->
      <!-- rpy values are chosen so the x and z axes are consistent with the internal sensor measurement frame -->
       <origin xyz="-0.0935 0 -0.0767" rpy="${pi} 0 ${pi/2}" />
       <parent link="${prefix}base_link" />
-      <child link="${prefix}aperture_frame" />
+      <child link="${prefix}optical_frame" />
     </joint>
   </xacro:macro>
